Commit message: Update launch files to use xacro --inorder.

File: urdf/apriltag_demo.xacro (robot description, xacro)
@@ -12,11 +12,11 @@
     <child  link="doro/world" />
   </joint>
-  <xacro:apriltag_marker namespace="doro/" name="apriltag1" parent="world" family="36h11" ID="1" size="0.5">
+  <xacro:apriltag_marker namespace="doro/" name="apriltag1" parent="world" family="36_11" ID="333" size="0.5">
     <origin xyz="1 1 1" rpy=" 0 0 0" />
   </xacro:apriltag_marker>
-  <xacro:apriltag_marker namespace="doro/" name="apriltag2" parent="world" family="36h11" ID="2" size="0.1">
+  <xacro:apriltag_marker namespace="doro/" name="apriltag2" parent="world" family="16_05" ID="2" size="0.1">
     <origin xyz="0.5 1 1" rpy=" 0 0 0" />
   </xacro:apriltag_marker>
-  <xacro:apriltag_marker namespace="doro/" name="apriltag3" parent="world" family="36h11" ID="3" size="0.1">
+  <xacro:apriltag_marker namespace="doro/" name="apriltag3" parent="world" family="36_11" ID="586" size="0.1">
     <origin xyz="0.5 0.5 1" rpy=" 0 0 0.8" />
   </xacro:apriltag_marker>

File: urdf/apriltag_marker.xacro (robot description, xacro)
@@ -10,9 +10,10 @@
        The marker is centered and can be added to other xacro/urdf
        models.
+       2019.05.22 - switch to textured Collada meshes, needs Jade or higher
        2014.11.24 - created
        (C) 2014 fnh, hendrich@informatik.uni-hamburg.de
        Usage:
        <xacro:apriltag_marker namespace="doro/" name="apriltag13" parent="base_link"
-              family="36h11" ID="13" size="0.05">
+              family="36_11" ID="00013" size="0.05">
          <origin xyz="0.2 0.3 05" rpy="0 0 3.14" />
        </xacro:apriltag_marker>
@@ -32,19 +33,13 @@
       </collision>
       <visual>
-        <!--<material name="red" />-->
         <origin xyz="0 0 0" rpy="0 0 1.571" />
         <geometry>
-          <box size="${size} ${size} 0.001" />
+          <!-- use Python str to convert family name and to generate leading zeros -->
+          <mesh filename="package://tams_apriltags/meshes/tag${str(family).replace( 'h', '_' )}_${str(ID).zfill(5)}.dae" scale="${10*size} ${10*size} 1"/>
         </geometry>
-        <material name="apriltag_${family}/tag${family}_${ID}" >
-        <!-- we generate 5-digit numbers in the filenames; for 36h11 this means we need 2 leading zeros -->
-        <!--<texture filename="file://$(find tams_apriltags)/Media/materials/textures/tag${family}/tag36_11_0000${ID}.png" />-->
-	        <texture filename="file://$(find tams_apriltags)/Media/materials/textures/rviz/${family}/${ID}.png" />
-        </material>
       </visual>
     </link>
     <!-- we use Gazebo material to put the texture onto the marker. Note mu1=mu2=0 for no friction. -->
     <gazebo reference="${namespace}${name}">
-      <material>apriltag_${family}/tag${family}_${ID}</material>
       <!-- <material>Gazebo/Red</material> -->
       <turnGravityOff>false</turnGravityOff>
