Commit message: Add 16h5 tag to the demo; update size of the cubes.

File: urdf/april_cube_40.xacro (robot description, xacro)
@@ -8,10 +8,10 @@
   <!-- note that our apriltag textures include the white border around
        the actual pattern (100x100 pixels total, with 80x80 pixels pattern).
-       For example, our demo cubes are 70x70x70 mm diameter, and this
+       For example, our demo cubes are 72x72x72 mm diameter, and this
        needs to be specified here for marker_size. The apriltags node
-       instead want the "internal" size, which is 0.056 (0.07*80/100)
+       instead want the "internal" size, which is 0.058 (0.072*80/100)
        in this case.
   -->
-  <xacro:april_cube name="april_cube_40" size="0.07" marker_size="0.07"
+  <xacro:april_cube name="april_cube_40" size="0.072" marker_size="0.072"
       id_top="40" id_front="41" id_right="42" id_back="43" id_left="44" id_bottom="45" />
 </robot>

File: urdf/april_cube_46.xacro (robot description, xacro)
@@ -8,10 +8,10 @@
   <!-- note that our apriltag textures include the white border around
        the actual pattern (100x100 pixels total, with 80x80 pixels pattern).
-       For example, our demo cubes are 70x70x70 mm diameter, and this
+       For example, our demo cubes are 72x72x72 mm diameter, and this
        needs to be specified here for marker_size. The apriltags node
-       instead want the "internal" size, which is 0.056 (0.07*80/100)
+       instead want the "internal" size, which is 0.058 (0.07*80/100)
        in this case.
   -->
-  <xacro:april_cube name="april_cube_46" size="0.07" marker_size="0.07"
+  <xacro:april_cube name="april_cube_46" size="0.072" marker_size="0.072"
       id_top="46" id_front="47" id_right="48" id_back="49" id_left="50" id_bottom="51" />
 </robot>

File: urdf/april_cube_60.xacro (robot description, xacro)
@@ -8,10 +8,10 @@
   <!-- note that our apriltag textures include the white border around
        the actual pattern (100x100 pixels total, with 80x80 pixels pattern).
-       For example, our demo cubes are 70x70x70 mm diameter, and this
+       For example, our demo cubes are 72x72x72 mm diameter, and this
        needs to be specified here for marker_size. The apriltags node
-       instead want the "internal" size, which is 0.056 (0.07*80/100)
+       instead want the "internal" size, which is 0.058 (0.072*80/100)
        in this case.
   -->
-  <xacro:april_cube name="april_cube_60" size="0.07" marker_size="0.07"
+  <xacro:april_cube name="april_cube_60" size="0.072" marker_size="0.072"
       id_top="60" id_front="61" id_right="62" id_back="63" id_left="64" id_bottom="65" />
 </robot>

File: urdf/apriltag_demo.xacro (robot description, xacro)
@@ -21,3 +21,6 @@
     <origin xyz="0.5 0.5 1" rpy=" 0 0 0.8" />
   </xacro:apriltag_marker>
+  <xacro:apriltag_marker namespace="doro/" name="apriltag4" parent="world" family="16_05" ID="23" size="0.1">
+    <origin xyz="0.25 0.25 1" rpy=" 0 0 0.7" />
+  </xacro:apriltag_marker>
 </robot>

Commit message: Remove outdated playerstage xmlns definitions.

File: urdf/april_cube_40.xacro (robot description, xacro)
@@ -1,7 +1,4 @@
 <?xml version="1.0" ?>
-<robot xmlns:sensor="http://playerstage.sourceforge.net/gazebo/xmlschema/#sensor"
-       xmlns:controller="http://playerstage.sourceforge.net/gazebo/xmlschema/#controller"
-       xmlns:interface="http://playerstage.sourceforge.net/gazebo/xmlschema/#interface"
-       xmlns:xacro="http://www.ros.org/wiki/xacro"
+<robot xmlns:xacro="http://www.ros.org/wiki/xacro"
        name="april_cube_40">
   <xacro:include filename="$(find tams_apriltags)/urdf/april_cube.xacro" />

File: urdf/april_cube_46.xacro (robot description, xacro)
@@ -1,7 +1,4 @@
 <?xml version="1.0" ?>
-<robot xmlns:sensor="http://playerstage.sourceforge.net/gazebo/xmlschema/#sensor"
-       xmlns:controller="http://playerstage.sourceforge.net/gazebo/xmlschema/#controller"
-       xmlns:interface="http://playerstage.sourceforge.net/gazebo/xmlschema/#interface"
-       xmlns:xacro="http://www.ros.org/wiki/xacro"
+<robot xmlns:xacro="http://www.ros.org/wiki/xacro"
        name="april_cube_46">
   <xacro:include filename="$(find tams_apriltags)/urdf/april_cube.xacro" />

File: urdf/april_cube_52.xacro (robot description, xacro)
@@ -1,7 +1,4 @@
 <?xml version="1.0" ?>
-<robot xmlns:sensor="http://playerstage.sourceforge.net/gazebo/xmlschema/#sensor"
-       xmlns:controller="http://playerstage.sourceforge.net/gazebo/xmlschema/#controller"
-       xmlns:interface="http://playerstage.sourceforge.net/gazebo/xmlschema/#interface"
-       xmlns:xacro="http://www.ros.org/wiki/xacro"
+<robot xmlns:xacro="http://www.ros.org/wiki/xacro"
        name="april_cube_52">
   <xacro:include filename="$(find tams_apriltags)/urdf/april_cube.xacro" />

File: urdf/april_cube_60.xacro (robot description, xacro)
@@ -1,7 +1,4 @@
 <?xml version="1.0" ?>
-<robot xmlns:sensor="http://playerstage.sourceforge.net/gazebo/xmlschema/#sensor"
-       xmlns:controller="http://playerstage.sourceforge.net/gazebo/xmlschema/#controller"
-       xmlns:interface="http://playerstage.sourceforge.net/gazebo/xmlschema/#interface"
-       xmlns:xacro="http://www.ros.org/wiki/xacro"
+<robot xmlns:xacro="http://www.ros.org/wiki/xacro"
        name="april_cube_60">
   <xacro:include filename="$(find tams_apriltags)/urdf/april_cube.xacro" />

File: urdf/april_cube_demo.xacro (robot description, xacro)
@@ -1,7 +1,4 @@
 <?xml version="1.0" ?>
-<robot xmlns:sensor="http://playerstage.sourceforge.net/gazebo/xmlschema/#sensor"
-       xmlns:controller="http://playerstage.sourceforge.net/gazebo/xmlschema/#controller"
-       xmlns:interface="http://playerstage.sourceforge.net/gazebo/xmlschema/#interface"
-       xmlns:xacro="http://www.ros.org/wiki/xacro"
+<robot xmlns:xacro="http://www.ros.org/wiki/xacro"
        name="apriltag_demo">
   <xacro:include filename="$(find tams_apriltags)/urdf/april_cube.xacro" />

File: urdf/apriltag_demo.xacro (robot description, xacro)
@@ -1,7 +1,4 @@
 <?xml version="1.0" ?>
-<robot xmlns:sensor="http://playerstage.sourceforge.net/gazebo/xmlschema/#sensor"
-       xmlns:controller="http://playerstage.sourceforge.net/gazebo/xmlschema/#controller"
-       xmlns:interface="http://playerstage.sourceforge.net/gazebo/xmlschema/#interface"
-       xmlns:xacro="http://www.ros.org/wiki/xacro"
+<robot xmlns:xacro="http://www.ros.org/wiki/xacro"
        name="apriltag_demo">
   <xacro:include filename="$(find tams_apriltags)/urdf/apriltag_marker.xacro" />

File: urdf/apriltag_marker.xacro (robot description, xacro)
@@ -1,7 +1,4 @@
 <?xml version="1.0" ?>
-<robot xmlns:sensor="http://playerstage.sourceforge.net/gazebo/xmlschema/#sensor"
-       xmlns:controller="http://playerstage.sourceforge.net/gazebo/xmlschema/#controller"
-       xmlns:interface="http://playerstage.sourceforge.net/gazebo/xmlschema/#interface"
-       xmlns:xacro="http://www.ros.org/wiki/xacro"
+<robot xmlns:xacro="http://www.ros.org/wiki/xacro"
        name="apriltag_marker">
   <!-- ROS xacro/urdf model of one apriltag marker with given
@@ -25,5 +22,5 @@
         <mass value="0.001" />
         <origin xyz="0 0 0" rpy="0 0 0" />
-        <inertia ixx="0.01" ixy="0" ixz="0" iyy="0.01" iyz="0" izz="0.01" />
+        <inertia ixx="0.00001" ixy="0" ixz="0" iyy="0.00001" iyz="0" izz="0.00002" />
       </inertial>
       <collision>

File: urdf/hanoi_demo.xacro (robot description, xacro)
@@ -1,7 +1,4 @@
 <?xml version="1.0" ?>
-<robot xmlns:sensor="http://playerstage.sourceforge.net/gazebo/xmlschema/#sensor"
-       xmlns:controller="http://playerstage.sourceforge.net/gazebo/xmlschema/#controller"
-       xmlns:interface="http://playerstage.sourceforge.net/gazebo/xmlschema/#interface"
-       xmlns:xacro="http://www.ros.org/wiki/xacro"
+<robot xmlns:xacro="http://www.ros.org/wiki/xacro"
        name="apriltag_demo">
   <xacro:include filename="$(find tams_apriltgas)/urdf/apriltag_marker.xacro" />

File: urdf/phasespace_calibration_board.xacro (robot description, xacro)
@@ -1,8 +1,4 @@
 <?xml version="1.0" ?>
-<robot
-       xmlns:sensor="http://playerstage.sourceforge.net/gazebo/xmlschema/#sensor"
-       xmlns:controller="http://playerstage.sourceforge.net/gazebo/xmlschema/#controller"
-       xmlns:interface="http://playerstage.sourceforge.net/gazebo/xmlschema/#interface"
-       xmlns:xacro="http://www.ros.org/wiki/xacro"
+<robot xmlns:xacro="http://www.ros.org/wiki/xacro"
        name="phasespace_calibration_board">
   <!-- a foam cube of given size with one centered apriltag of given

File: urdf/phasespace_calibration_board_instance.xacro (robot description, xacro)
@@ -1,7 +1,4 @@
 <?xml version="1.0" ?>
-<robot xmlns:sensor="http://playerstage.sourceforge.net/gazebo/xmlschema/#sensor"
-       xmlns:controller="http://playerstage.sourceforge.net/gazebo/xmlschema/#controller"
-       xmlns:interface="http://playerstage.sourceforge.net/gazebo/xmlschema/#interface"
-       xmlns:xacro="http://www.ros.org/wiki/xacro"
+<robot xmlns:xacro="http://www.ros.org/wiki/xacro"
        name="phasespace_calibration_demo">
   <!-- a foam cube of given size with one centered apriltag of given

File: urdf/phasespace_calibration_demo.xacro (robot description, xacro)
@@ -1,7 +1,4 @@
 <?xml version="1.0" ?>
-<robot xmlns:sensor="http://playerstage.sourceforge.net/gazebo/xmlschema/#sensor"
-       xmlns:controller="http://playerstage.sourceforge.net/gazebo/xmlschema/#controller"
-       xmlns:interface="http://playerstage.sourceforge.net/gazebo/xmlschema/#interface"
-       xmlns:xacro="http://www.ros.org/wiki/xacro"
+<robot xmlns:xacro="http://www.ros.org/wiki/xacro"
        name="phasespace_calibration_demo">
   <!-- a foam cube of given size with one centered apriltag of given

File: urdf/thiago_cards_demo.xacro (robot description, xacro)
@@ -1,7 +1,4 @@
 <?xml version="1.0" ?>
-<robot xmlns:sensor="http://playerstage.sourceforge.net/gazebo/xmlschema/#sensor"
-       xmlns:controller="http://playerstage.sourceforge.net/gazebo/xmlschema/#controller"
-       xmlns:interface="http://playerstage.sourceforge.net/gazebo/xmlschema/#interface"
-       xmlns:xacro="http://www.ros.org/wiki/xacro"
+<robot xmlns:xacro="http://www.ros.org/wiki/xacro"
        name="apriltag_demo">
   <xacro:include filename="$(find tams_apriltags)/urdf/thiago_command_card.xacro" />

File: urdf/thiago_command_card.xacro (robot description, xacro)
@@ -1,7 +1,4 @@
 <?xml version="1.0" ?>
-<robot xmlns:sensor="http://playerstage.sourceforge.net/gazebo/xmlschema/#sensor"
-       xmlns:controller="http://playerstage.sourceforge.net/gazebo/xmlschema/#controller"
-       xmlns:interface="http://playerstage.sourceforge.net/gazebo/xmlschema/#interface"
-       xmlns:xacro="http://www.ros.org/wiki/xacro"
+<robot xmlns:xacro="http://www.ros.org/wiki/xacro"
        name="thiago_card">
   <!-- ROS xacro/urdf model of one "Thiago demo command card",

File: urdf/tiago_cards_demo.xacro (robot description, xacro)
@@ -1,7 +1,4 @@
 <?xml version="1.0" ?>
-<robot xmlns:sensor="http://playerstage.sourceforge.net/gazebo/xmlschema/#sensor"
-       xmlns:controller="http://playerstage.sourceforge.net/gazebo/xmlschema/#controller"
-       xmlns:interface="http://playerstage.sourceforge.net/gazebo/xmlschema/#interface"
-       xmlns:xacro="http://www.ros.org/wiki/xacro"
+<robot xmlns:xacro="http://www.ros.org/wiki/xacro"
        name="apriltag_demo">
   <xacro:include filename="$(find tams_apriltags)/urdf/tiago_command_card.xacro" />

File: urdf/tiago_command_card.xacro (robot description, xacro)
@@ -1,7 +1,4 @@
 <?xml version="1.0" ?>
-<robot xmlns:sensor="http://playerstage.sourceforge.net/gazebo/xmlschema/#sensor"
-       xmlns:controller="http://playerstage.sourceforge.net/gazebo/xmlschema/#controller"
-       xmlns:interface="http://playerstage.sourceforge.net/gazebo/xmlschema/#interface"
-       xmlns:xacro="http://www.ros.org/wiki/xacro"
+<robot xmlns:xacro="http://www.ros.org/wiki/xacro"
        name="tiago_card">
   <!-- ROS xacro/urdf model of one "Tiago demo command card",

File: urdf/utilities.xacro (robot description, xacro)
@@ -1,8 +1,5 @@
 <?xml version="1.0"?>
-<robot xmlns:sensor="http://playerstage.sourceforge.net/gazebo/xmlschema/#sensor"
-   xmlns:controller="http://playerstage.sourceforge.net/gazebo/xmlschema/#controller"
-   xmlns:interface="http://playerstage.sourceforge.net/gazebo/xmlschema/#interface"
-   xmlns:xacro="http://playerstage.sourceforge.net/gazebo/xmlschema/#interface"
-   name="utilities">
+<robot xmlns:xacro="http://www.ros.org/wiki/xacro"
+       name="utilities">
 <!-- idea and easy_box borrowed from B21.xacro,
      <url>http://ros.org/wiki/b21_description</url>, BSD license
