Commit message: Fix wrong marker rotation.

File: urdf/apriltag_marker.xacro (robot description, xacro)
@@ -10,4 +10,5 @@
        The marker is centered and can be added to other xacro/urdf
        models.
+       2019.10.10 - fix Collada rotation, ooops
        2019.05.22 - switch to textured Collada meshes, needs Jade or higher
        2014.11.24 - created
@@ -27,5 +28,5 @@
       </inertial>
       <collision>
-        <origin xyz="0 0 0" rpy="0 0 1.571" />
+        <origin xyz="0 0 0" rpy="0 0 0" />
         <geometry>
           <box size="${size} ${size} 0.001" />
@@ -33,5 +34,5 @@
       </collision>
       <visual>
-        <origin xyz="0 0 0" rpy="0 0 1.571" />
+        <origin xyz="0 0 0" rpy="0 0 0" />
         <geometry>
           <!-- use Python str to convert family name and to generate leading zeros -->

Commit message: Add parameter to specify marker/apriltag size
With the parameter ""include_borders":=false" it is possible to specify
whether the desired size is the size of the whole marker including borders, or
just of the apriltag marker. In the latter case the size of the resulting
marker will be bigger due to the mandatory white borders around the
apriltag

File: urdf/apriltag_marker.xacro (robot description, xacro)
@@ -7,15 +7,36 @@
        The marker is centered and can be added to other xacro/urdf
        models.
+       The parameter "include_borders" is used to indicate
+       whether the one bit wide white borders are included in the
+       size specification. If "include_borders" is set to true,
+       the actual size of the apriltag will be:
+       8/10*size in case of 36h11
+       6/8 *size in case of 16h5
+       This is due to the usage of the white border in the
+       apriltag detection algorithm, even though its size
+       is not specified.
        2019.10.10 - fix Collada rotation, ooops
        2019.05.22 - switch to textured Collada meshes, needs Jade or higher
        2014.11.24 - created
+       2021.11.10 - added include_borders parameter
        (C) 2014 fnh, hendrich@informatik.uni-hamburg.de
        Usage:
        <xacro:apriltag_marker namespace="doro/" name="apriltag13" parent="base_link"
-              family="36_11" ID="00013" size="0.05">
+              family="36h11" ID="00013" size="0.05" include_borders="false">
          <origin xyz="0.2 0.3 05" rpy="0 0 3.14" />
        </xacro:apriltag_marker>
    -->
-  <xacro:macro name="apriltag_marker" params="namespace name parent family ID size *origin" >
+  <xacro:macro name="apriltag_marker" params="namespace name parent family ID size include_borders:=true *origin" >
+    <xacro:if value="${include_borders == False}">
+      <xacro:if value="${family == '36h11'}">
+        <xacro:property name="mesh_size" value="${size/8*10}" />
+      </xacro:if>
+      <xacro:if value="${family == '16h5'}">
+        <xacro:property name="mesh_size" value="${size/6*8}" />
+      </xacro:if>
+    </xacro:if>
+    <xacro:if value="${include_borders == True}">
+      <xacro:property name="mesh_size" value="${size}" />
+    </xacro:if>
     <link name="${namespace}${name}">
       <inertial>
@@ -27,5 +48,5 @@
         <origin xyz="0 0 0" rpy="0 0 0" />
         <geometry>
-          <box size="${size} ${size} 0.001" />
+          <box size="${mesh_size} ${mesh_size} 0.001" />
         </geometry>
       </collision>
@@ -34,5 +55,5 @@
         <geometry>
           <!-- use Python str to convert family name and to generate leading zeros -->
-          <mesh filename="package://tams_apriltags/meshes/tag${str(family).replace( 'h', '_' )}_${str(ID).zfill(5)}.dae" scale="${10*size} ${10*size} 1"/>
+          <mesh filename="package://tams_apriltags/meshes/tag${str(family).replace( 'h', '_' )}_${str(ID).zfill(5)}.dae" scale="${10*mesh_size} ${10*mesh_size} 1"/>
         </geometry>
       </visual>

Commit message: Change interface of the april_tag macro
Now takes size of the mesh or size of the april tag

File: urdf/apriltag_marker.xacro (robot description, xacro)
@@ -3,11 +3,11 @@
        name="apriltag_marker">
   <!-- ROS xacro/urdf model of one apriltag marker with given
-       tag-family, ID, and size. The marker is modeled as a simple
-       box with outer xy diameter as specified, and z 1mm thickness.
+       tag-family, ID, and size of the mesh. Optionally, apriltag_size can be
+       specified to calculate from it the size of the mesh. In this case the
+       parameter "size" will be ignored. The marker is modeled as
+       a simple box with outer xy diameter as specified, and z 1mm thickness.
        The marker is centered and can be added to other xacro/urdf
        models.
-       The parameter "include_borders" is used to indicate
-       whether the one bit wide white borders are included in the
-       size specification. If "include_borders" is set to true,
+       The mesh of the model contains one bit wide white borders. Therefore,
        the actual size of the apriltag will be:
        8/10*size in case of 36h11
@@ -15,5 +15,5 @@
        This is due to the usage of the white border in the
        apriltag detection algorithm, even though its size
-       is not specified.
+       does not have a convention.
        2019.10.10 - fix Collada rotation, ooops
        2019.05.22 - switch to textured Collada meshes, needs Jade or higher
@@ -22,4 +22,7 @@
        (C) 2014 fnh, hendrich@informatik.uni-hamburg.de
        Usage:
+       size - size of the mesh
+       apriltag_size - size of the apriltag. If this parameter is set, the size
+       of the mesh will be re-calculated
        <xacro:apriltag_marker namespace="doro/" name="apriltag13" parent="base_link"
               family="36h11" ID="00013" size="0.05" include_borders="false">
@@ -27,6 +30,9 @@
        </xacro:apriltag_marker>
    -->
-  <xacro:macro name="apriltag_marker" params="namespace name parent family ID size include_borders:=true *origin" >
-    <xacro:if value="${include_borders == False}">
+  <xacro:macro name="apriltag_marker" params="namespace name parent family ID size apriltag_size:=-1 *origin" >
+    <xacro:if value="${apriltag_size == -1}">
+      <xacro:property name="mesh_size" value="${apriltag_size}" />
+    </xacro:if>
+    <xacro:if value="${apriltag_size != -1}">
       <xacro:if value="${family == '36h11'}">
         <xacro:property name="mesh_size" value="${size/8*10}" />
@@ -35,7 +41,4 @@
         <xacro:property name="mesh_size" value="${size/6*8}" />
       </xacro:if>
-    </xacro:if>
-    <xacro:if value="${include_borders == True}">
-      <xacro:property name="mesh_size" value="${size}" />
     </xacro:if>
     <link name="${namespace}${name}">

Commit message: Add default value, correct bug with function interface

File: urdf/apriltag_marker.xacro (robot description, xacro)
@@ -30,14 +30,14 @@
        </xacro:apriltag_marker>
    -->
-  <xacro:macro name="apriltag_marker" params="namespace name parent family ID size apriltag_size:=-1 *origin" >
-    <xacro:if value="${apriltag_size == -1}">
-      <xacro:property name="mesh_size" value="${apriltag_size}" />
+  <xacro:macro name="apriltag_marker" params="namespace name parent family ID size:=0 apriltag_size:=0 *origin" >
+    <xacro:if value="${apriltag_size == 0}">
+      <xacro:property name="mesh_size" value="${size}" />
     </xacro:if>
-    <xacro:if value="${apriltag_size != -1}">
+    <xacro:if value="${apriltag_size != 0}">
       <xacro:if value="${family == '36h11'}">
-        <xacro:property name="mesh_size" value="${size/8*10}" />
+        <xacro:property name="mesh_size" value="${apriltag_size/8*10}" />
       </xacro:if>
       <xacro:if value="${family == '16h5'}">
-        <xacro:property name="mesh_size" value="${size/6*8}" />
+        <xacro:property name="mesh_size" value="${apriltag_size/6*8}" />
       </xacro:if>
     </xacro:if>

Commit message: Change readme

File: urdf/apriltag_marker.xacro (robot description, xacro)
@@ -4,5 +4,5 @@
   <!-- ROS xacro/urdf model of one apriltag marker with given
        tag-family, ID, and size of the mesh. Optionally, apriltag_size can be
-       specified to calculate from it the size of the mesh. In this case the
+       specified to calculate from it the size of the mesh. In this case, the
        parameter "size" will be ignored. The marker is modeled as
        a simple box with outer xy diameter as specified, and z 1mm thickness.
@@ -24,11 +24,22 @@
        size - size of the mesh
        apriltag_size - size of the apriltag. If this parameter is set, the size
-       of the mesh will be re-calculated
+       of the mesh will be re-calculated as mentioned above
        <xacro:apriltag_marker namespace="doro/" name="apriltag13" parent="base_link"
-              family="36h11" ID="00013" size="0.05" include_borders="false">
+              family="36h11" ID="00013" size="0.33" >
+         <origin xyz="0.2 0.3 05" rpy="0 0 3.14" />
+       <xacro:apriltag_marker namespace="doro/" name="apriltag14" parent="base_link"
+              family="36h11" ID="00014" apriltag_size="0.5">
+         <origin xyz="0.2 0.3 05" rpy="0 0 3.14" />
+       </xacro:apriltag_marker>
+       The following definition does not make much sense and will produce the same result
+       as the one above with ID=00014, because the mesh is predefined and the size of the
+       border will not be recalculated.
+       <xacro:apriltag_marker namespace="doro/" name="apriltag14" parent="base_link"
+              family="36h11" ID="00014" size="0.33" apriltag_size="0.5">
          <origin xyz="0.2 0.3 05" rpy="0 0 3.14" />
        </xacro:apriltag_marker>
    -->
   <xacro:macro name="apriltag_marker" params="namespace name parent family ID size:=0 apriltag_size:=0 *origin" >
+    <!-- Check in which way the size was specified -->
     <xacro:if value="${apriltag_size == 0}">
       <xacro:property name="mesh_size" value="${size}" />

Commit message: Add parameter to specify marker/apriltag size (#1)
Co-authored-by: Mykhailo Koshil <mykhailo.koshil@gmail.com>

File: urdf/apriltag_marker.xacro (robot description, xacro)
@@ -3,19 +3,54 @@
        name="apriltag_marker">
   <!-- ROS xacro/urdf model of one apriltag marker with given
-       tag-family, ID, and size. The marker is modeled as a simple
-       box with outer xy diameter as specified, and z 1mm thickness.
+       tag-family, ID, and size of the mesh. Optionally, apriltag_size can be
+       specified to calculate from it the size of the mesh. In this case, the
+       parameter "size" will be ignored. The marker is modeled as
+       a simple box with outer xy diameter as specified, and z 1mm thickness.
        The marker is centered and can be added to other xacro/urdf
        models.
+       The mesh of the model contains one bit wide white borders. Therefore,
+       the actual size of the apriltag will be:
+       8/10*size in case of 36h11
+       6/8 *size in case of 16h5
+       This is due to the usage of the white border in the
+       apriltag detection algorithm, even though its size
+       does not have a convention.
        2019.10.10 - fix Collada rotation, ooops
        2019.05.22 - switch to textured Collada meshes, needs Jade or higher
        2014.11.24 - created
+       2021.11.10 - added include_borders parameter
        (C) 2014 fnh, hendrich@informatik.uni-hamburg.de
        Usage:
+       size - size of the mesh
+       apriltag_size - size of the apriltag. If this parameter is set, the size
+       of the mesh will be re-calculated as mentioned above
        <xacro:apriltag_marker namespace="doro/" name="apriltag13" parent="base_link"
-              family="36_11" ID="00013" size="0.05">
+              family="36h11" ID="00013" size="0.33" >
+         <origin xyz="0.2 0.3 05" rpy="0 0 3.14" />
+       <xacro:apriltag_marker namespace="doro/" name="apriltag14" parent="base_link"
+              family="36h11" ID="00014" apriltag_size="0.05">
+         <origin xyz="0.2 0.3 05" rpy="0 0 3.14" />
+       </xacro:apriltag_marker>
+       The following definition does not make much sense and will produce the same result
+       as the one above with ID=00014, because the mesh is predefined and the size of the
+       border will not be recalculated.
+       <xacro:apriltag_marker namespace="doro/" name="apriltag14" parent="base_link"
+              family="36h11" ID="00014" size="0.33" apriltag_size="0.05">
          <origin xyz="0.2 0.3 05" rpy="0 0 3.14" />
        </xacro:apriltag_marker>
    -->
-  <xacro:macro name="apriltag_marker" params="namespace name parent family ID size *origin" >
+  <xacro:macro name="apriltag_marker" params="namespace name parent family ID size:=0 apriltag_size:=0 *origin" >
+    <!-- Check in which way the size was specified -->
+    <xacro:if value="${apriltag_size == 0}">
+      <xacro:property name="mesh_size" value="${size}" />
+    </xacro:if>
+    <xacro:if value="${apriltag_size != 0}">
+      <xacro:if value="${family == '36h11'}">
+        <xacro:property name="mesh_size" value="${apriltag_size/8*10}" />
+      </xacro:if>
+      <xacro:if value="${family == '16h5'}">
+        <xacro:property name="mesh_size" value="${apriltag_size/6*8}" />
+      </xacro:if>
+    </xacro:if>
     <link name="${namespace}${name}">
       <inertial>
@@ -27,5 +62,5 @@
         <origin xyz="0 0 0" rpy="0 0 0" />
         <geometry>
-          <box size="${size} ${size} 0.001" />
+          <box size="${mesh_size} ${mesh_size} 0.001" />
         </geometry>
       </collision>
@@ -34,5 +69,5 @@
         <geometry>
           <!-- use Python str to convert family name and to generate leading zeros -->
-          <mesh filename="package://tams_apriltags/meshes/tag${str(family).replace( 'h', '_' )}_${str(ID).zfill(5)}.dae" scale="${10*size} ${10*size} 1"/>
+          <mesh filename="package://tams_apriltags/meshes/tag${str(family).replace( 'h', '_' )}_${str(ID).zfill(5)}.dae" scale="${10*mesh_size} ${10*mesh_size} 1"/>
         </geometry>
       </visual>
